File: Hardware/KiCad-Files/Main_board/Main_board.kicad_sch (KiCad schematic)
At the start: 46 parts, among them Q1 MOSFET-NGDS_TO220V, U1 ESP32-DEVKITC-32D, X1 W237-102

Commit message: Another update
Parts:
- removed U$2: BUCK_MODULEWITH_SMDPADS&THROUGHHOLES, WK_Samec-12pin:Buck_Converter, symbol Main_board-eagle-import:BUCK_MODULEWITH_SMDPADS&THROUGHHOLES
- added U3: Buck_converter-LM2596, symbol Buck_Converter:Buck_converter-LM2596
- Q1: value MOSFET-NGDS_TO220V -> N-MOSFET
- renumbered U$1 to U2, SV1 to X2, SV5 to X3, SV2 to X4-1, SV3 to X4-2, SV4 to X4-3
Connections:
- net GND2 is gone; now on net GND: U1.26 (GND2)
- net GND: now also C4.2, C5.1, JP5.1, R8.1, U2.2 (GND), X2.10, X2.11, X2.12, U3.2 (IN-), U3.3 (OUT-)
- net at X2.1, X2.2, X2.3: now also F1.2; no longer F1.1
- net at C4.1, D3.C, JP4.1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: now also F1.1; no longer F1.2
- net at X4-2.2, X4-2.4, X4-3.2: now also X4-1.2, X4-1.4
- net at D1.C, D2.C: now also U3.1 (IN+)
- net at D3.A: now also U3.4 (OUT+)
Other:
- moved on the sheet: C1, C2, C3, C4, C5, D3, F1, JP1, JP2, JP3, JP4, JP5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
