File: Hardware/KiCad-Files/Home_Unit_OLED/Home_Unit_OLED.kicad_sch (KiCad schematic)
At the start: 14 parts, among them J1 Conn_01x02, J2 Conn_01x06, J3 Conn_01x04, SW1 FLASH, SW2 RESET, U1 AMS1117-3.3, U2 ESP-12S

Commit message: Update
Parts:
- renumbered J1 to X1, J2 to X2, J3 to X3
Changed lines of the file:
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@@
   (symbol (lib_id "Connector_Generic:Conn_01x06") (at 204.47 59.69 0) (unit 1)
     (in_bom yes) (on_board yes) (fields_autoplaced)
-    (property "Reference" "J2" (id 0) (at 207.01 59.6899 0)
+    (property "Reference" "X2" (id 0) (at 207.01 59.6899 0)
       (effects (font (size 1.27 1.27)) (justify left))
     )
@@
   (symbol (lib_id "Connector_Generic:Conn_01x02") (at 71.12 110.49 0) (mirror y) (unit 1)
     (in_bom yes) (on_board yes) (fields_autoplaced)
-    (property "Reference" "J1" (id 0) (at 71.12 104.14 0))
+    (property "Reference" "X1" (id 0) (at 71.12 104.14 0))
     (property "Value" "Conn_01x02" (id 1) (at 71.12 106.68 0))
     (property "Footprint" "" (id 2) (at 71.12 110.49 0)
@@
   (symbol (lib_id "Connector_Generic:Conn_01x04") (at 219.71 74.93 0) (unit 1)
     (in_bom yes) (on_board yes) (fields_autoplaced)
-    (property "Reference" "J3" (id 0) (at 222.25 74.9299 0)
+    (property "Reference" "X3" (id 0) (at 222.25 74.9299 0)
       (effects (font (size 1.27 1.27)) (justify left))
     )
@@
       (reference "C2") (unit 1) (value "100n") (footprint "")
     )
-    (path "/92202be8-5406-4a1d-bf47-5cd2538fcd51"
-      (reference "J1") (unit 1) (value "Conn_01x02") (footprint "")
-    )
-    (path "/74244b9c-c825-4f1a-8b96-f3b051d373b6"
-      (reference "J2") (unit 1) (value "Conn_01x06") (footprint "")
-    )
-    (path "/98406805-7176-44f6-971f-9a07303b0a80"
-      (reference "J3") (unit 1) (value "Conn_01x04") (footprint "")
-    )
     (path "/02ff3d26-cb04-42cd-9713-673e1faa89f1"
       (reference "R1") (unit 1) (value "10k") (footprint "")
@@
       (reference "U2") (unit 1) (value "ESP-12S") (footprint "ESP-12S")
     )
-  )
+    (path "/92202be8-5406-4a1d-bf47-5cd2538fcd51"
+      (reference "X1") (unit 1) (value "Conn_01x02") (footprint "")
+    )
+    (path "/74244b9c-c825-4f1a-8b96-f3b051d373b6"
+      (reference "X2") (unit 1) (value "Conn_01x06") (footprint "")
+    )
+    (path "/98406805-7176-44f6-971f-9a07303b0a80"
+      (reference "X3") (unit 1) (value "Conn_01x04") (footprint "")
+    )
+  )
