File: Hardware/KiCad-Files/Light_board/Light_board.kicad_sch (KiCad schematic)
At the start: 1 part

Commit message: Creating/modifying PCB and Schematic
Parts:
- removed J?: Conn_01x06_Male, Connector_PinHeader_2.54mm:PinHeader_1x06_P2.54mm_Vertical, symbol Connector:Conn_01x06_Male
- added A1: GYML-8511_ML8511, symbol GYML-8511_ML8511:GYML-8511_ML8511
- added A2: GY-302_BH1750, symbol GY-302_BH1750:GY-302_BH1750
- added J1: Conn_01x06, Connector_PinHeader_2.54mm:PinHeader_1x06_P2.54mm_Horizontal, symbol Connector_Generic:Conn_01x06
- added R1: GBR618, symbol GBR618-19:GBR618
Connections:
- new net: A2.2 (SDA), J1.2 (Pin_2)
- new net: A2.3 (SCL), J1.1 (Pin_1)
- new net: A1.2 (3V3), A1.5 (EN), A2.5 (VCC), J1.6 (Pin_6)
- new net: J1.3 (Pin_3), R1.
- new net: A1.4 (OUT), J1.4 (Pin_4)
- new net GND: A1.3 (GND), A2.4 (GND), J1.5 (Pin_5), R1.
Other:
- company: (none) -> Michal Basler
- title: (none) -> Deska pro měření světla a UV intenzity
Changed lines of the file:
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@@
 (kicad_sch (version 20211123) (generator eeschema)
   (paper "A4")
-  (symbol (lib_id "Connector:Conn_01x06_Male") (at 137.16 66.04 180) (unit 1)
+  (title_block
+    (title "Deska pro měření světla a UV intenzity")
+    (date "2022-03-02")
+    (rev "1.1")
+    (company "Michal Basler")
+    (comment 1 "Maturitní práce 2021/22")
+  )
+  (junction (at 166.37 119.38) (diameter 0) (color 0 0 0 0)
+  )
+  (junction (at 135.89 118.11) (diameter 0) (color 0 0 0 0)
+  )
+  (junction (at 127 118.11) (diameter 0) (color 0 0 0 0)
+  )
+  (junction (at 138.43 119.38) (diameter 0) (color 0 0 0 0)
+  )
+  (wire (pts (xy 163.83 113.03) (xy 163.83 127))
+    (stroke (width 0) (type default) (color 0 0 0 0))
+  )
+  (wire (pts (xy 119.38 118.11) (xy 119.38 113.03))
+    (stroke (width 0) (type default) (color 0 0 0 0))
+  )
+  (wire (pts (xy 138.43 119.38) (xy 121.92 119.38))
+    (stroke (width 0) (type default) (color 0 0 0 0))
+  )
+  (wire (pts (xy 138.43 119.38) (xy 138.43 127))
+    (stroke (width 0) (type default) (color 0 0 0 0))
+  )
+  (wire (pts (xy 127 113.03) (xy 127 118.11))
+    (stroke (width 0) (type default) (color 0 0 0 0))
+  )
+  (wire (pts (xy 135.89 118.11) (xy 135.89 127))
+    (stroke (width 0) (type default) (color 0 0 0 0))
+  )
+  (wire (pts (xy 140.97 127) (xy 140.97 116.84))
+    (stroke (width 0) (type default) (color 0 0 0 0))
+  )
+  (wire (pts (xy 161.29 124.46) (xy 161.29 113.03))
+    (stroke (width 0) (type default) (color 0 0 0 0))
+  )
+  (wire (pts (xy 168.91 113.03) (xy 168.91 118.11))
+    (stroke (width 0) (type default) (color 0 0 0 0))
+  )
+  (wire (pts (xy 135.89 118.11) (xy 127 118.11))
+    (stroke (width 0) (type default) (color 0 0 0 0))
+  )
+  (wire (pts (xy 163.83 127) (xy 148.59 127))
+    (stroke (width 0) (type default) (color 0 0 0 0))
+  )
+  (wire (pts (xy 121.92 119.38) (xy 121.92 113.03))
+    (stroke (width 0) (type default) (color 0 0 0 0))
+  )
+  (wire (pts (xy 146.05 124.46) (xy 161.29 124.46))
+    (stroke (width 0) (type default) (color 0 0 0 0))
+  )
+  (wire (pts (xy 148.59 114.3) (xy 148.59 111.76))
+    (stroke (width 0) (type default) (color 0 0 0 0))
+  )
+  (wire (pts (xy 143.51 127) (xy 143.51 114.3))
+    (stroke (width 0) (type default) (color 0 0 0 0))
+  )
+  (wire (pts (xy 135.89 118.11) (xy 168.91 118.11))
+    (stroke (width 0) (type default) (color 0 0 0 0))
+  )
+  (wire (pts (xy 143.51 114.3) (xy 148.59 114.3))
+    (stroke (width 0) (type default) (color 0 0 0 0))
+  )
+  (wire (pts (xy 127 118.11) (xy 119.38 118.11))
+    (stroke (width 0) (type default) (color 0 0 0 0))
+  )
+  (wire (pts (xy 140.97 116.84) (xy 124.46 116.84))
+    (stroke (width 0) (type default) (color 0 0 0 0))
+  )
+  (wire (pts (xy 166.37 119.38) (xy 138.43 119.38))
+    (stroke (width 0) (type default) (color 0 0 0 0))
+  )
+  (wire (pts (xy 124.46 116.84) (xy 124.46 113.03))
+    (stroke (width 0) (type default) (color 0 0 0 0))
+  )
+  (wire (pts (xy 138.43 111.76) (xy 138.43 119.38))
+    (stroke (width 0) (type default) (color 0 0 0 0))
+  )
+  (wire (pts (xy 146.05 127) (xy 146.05 124.46))
+    (stroke (width 0) (type default) (color 0 0 0 0))
+  )
+  (wire (pts (xy 166.37 113.03) (xy 166.37 119.38))
+    (stroke (width 0) (type default) (color 0 0 0 0))
+  )
+  (symbol (lib_id "power:GND") (at 166.37 119.38 0) (unit 1)
     (in_bom yes) (on_board yes) (fields_autoplaced)
-    (property "Reference" "J?" (id 0) (at 136.525 76.2 0))
-    (property "Value" "Conn_01x06_Male" (id 1) (at 136.525 73.66 0))
-    (property "Footprint" "Connector_PinHeader_2.54mm:PinHeader_1x06_P2.54mm_Vertical" (id 2) (at 137.16 66.04 0)
+    (property "Reference" "#PWR01" (id 0) (at 166.37 125.73 0)
       (effects (font (size 1.27 1.27)) hide)
     )
-    (property "Datasheet" "~" (id 3) (at 137.16 66.04 0)
+    (property "Value" "GND" (id 1) (at 166.37 124.46 0))
+    (property "Footprint" "" (id 2) (at 166.37 119.38 0)
+      (effects (font (size 1.27 1.27)) hide)
+    )
+    (property "Datasheet" "" (id 3) (at 166.37 119.38 0)
+      (effects (font (size 1.27 1.27)) hide)
+    )
+    (pin "1")
+  )
+  (symbol (lib_id "GY-302_BH1750:GY-302_BH1750") (at 163.83 110.49 0) (unit 1)
+    (in_bom yes) (on_board yes)
+    (property "Reference" "A2" (id 0) (at 172.72 104.7749 0)
+      (effects (font (size 1.27 1.27)) (justify left))
+    )
+    (property "Value" "GY-302_BH1750" (id 1) (at 156.21 100.33 0)
+      (effects (font (size 1.27 1.27)) (justify left))
+    )
+    (property "Footprint" "" (id 2) (at 163.83 99.06 0)
+      (effects (font (size 1.27 1.27)) hide)
+    )
+    (property "Datasheet" "" (id 3) (at 163.83 99.06 0)
+      (effects (font (size 1.27 1.27)) hide)
+    )
+    (pin "1")
+    (pin "2")
+    (pin "3")
+    (pin "4")
+    (pin "5")
+  )
+  (symbol (lib_id "GBR618-19:GBR618") (at 143.51 111.76 180) (unit 1)
+    (in_bom yes) (on_board yes) (fields_autoplaced)
+    (property "Reference" "R1" (id 0) (at 143.51 105.41 0))
+    (property "Value" "GBR618" (id 1) (at 143.51 107.95 0))
+    (property "Footprint" "" (id 2) (at 143.51 111.76 0)
+      (effects (font (size 1.27 1.27)) hide)
+    )
+    (property "Datasheet" "" (id 3) (at 143.51 111.76 0)
+      (effects (font (size 1.27 1.27)) hide)
+    )
+    (pin "")
+    (pin "")
+  )
+  (symbol (lib_id "GYML-8511_ML8511:GYML-8511_ML8511") (at 121.92 104.14 0) (unit 1)
+    (in_bom yes) (on_board yes)
+    (property "Reference" "A1" (id 0) (at 130.81 104.7749 0)
+      (effects (font (size 1.27 1.27)) (justify left))
+    )
+    (property "Value" "GYML-8511_ML8511" (id 1) (at 114.3 100.33 0)
+      (effects (font (size 1.27 1.27)) (justify left))
+    )
+    (property "Footprint" "" (id 2) (at 121.92 104.14 0)
+      (effects (font (size 1.27 1.27)) hide)
+    )
+    (property "Datasheet" "" (id 3) (at 121.92 104.14 0)
+      (effects (font (size 1.27 1.27)) hide)
+    )
+    (pin "1")
+    (pin "2")
+    (pin "3")
+    (pin "4")
+    (pin "5")
+  )
+  (symbol (lib_id "Connector_Generic:Conn_01x06") (at 143.51 132.08 270) (unit 1)
+    (in_bom yes) (on_board yes) (fields_autoplaced)
+    (property "Reference" "J1" (id 0) (at 142.24 135.89 90))
+    (property "Value" "Conn_01x06" (id 1) (at 142.24 138.43 90))
+    (property "Footprint" "Connector_PinHeader_2.54mm:PinHeader_1x06_P2.54mm_Horizontal" (id 2) (at 143.51 132.08 0)
+      (effects (font (size 1.27 1.27)) hide)
+    )
+    (property "Datasheet" "~" (id 3) (at 143.51 132.08 0)
       (effects (font (size 1.27 1.27)) hide)
     )
@@
   )
   (symbol_instances
-    (path "/edbc17dd-aa76-4d77-81ec-11ed42efea05"
-      (reference "J?") (unit 1) (value "Conn_01x06_Male") (footprint "Connector_PinHeader_2.54mm:PinHeader_1x06_P2.54mm_Vertical")
+    (path "/196e1018-3128-4152-8013-cccbdb3d095b"
+      (reference "#PWR01") (unit 1) (value "GND") (footprint "")
+    )
+    (path "/a5c3bc6f-0964-4788-98a2-3abcf65e12d1"
+      (reference "A1") (unit 1) (value "GYML-8511_ML8511") (footprint "")
+    )
+    (path "/2cd70291-d45b-4d51-a287-bd9d9781e2bc"
+      (reference "A2") (unit 1) (value "GY-302_BH1750") (footprint "")
+    )
+    (path "/d77d54ed-c281-49b8-a660-428ecc3d5c70"
+      (reference "J1") (unit 1) (value "Conn_01x06") (footprint "Connector_PinHeader_2.54mm:PinHeader_1x06_P2.54mm_Horizontal")
+    )
+    (path "/421acf1c-f4d2-4059-83d6-dfb83d6549e9"
+      (reference "R1") (unit 1) (value "GBR618") (footprint "")
     )
   )

Commit message: Update
Parts:
- R1_GBR-618: renamed from R1; value GBR618 -> 14.4R
- renumbered J1 to X1
Changed lines of the file:
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@@
   (symbol (lib_id "GBR618-19:GBR618") (at 143.51 111.76 180) (unit 1)
     (in_bom yes) (on_board yes) (fields_autoplaced)
-    (property "Reference" "R1" (id 0) (at 143.51 105.41 0))
-    (property "Value" "GBR618" (id 1) (at 143.51 107.95 0))
+    (property "Reference" "R1_GBR-618" (id 0) (at 143.51 105.41 0))
+    (property "Value" "14.4R" (id 1) (at 143.51 107.95 0))
     (property "Footprint" "" (id 2) (at 143.51 111.76 0)
       (effects (font (size 1.27 1.27)) hide)
@@
   (symbol (lib_id "Connector_Generic:Conn_01x06") (at 143.51 132.08 270) (unit 1)
     (in_bom yes) (on_board yes) (fields_autoplaced)
-    (property "Reference" "J1" (id 0) (at 142.24 135.89 90))
+    (property "Reference" "X1" (id 0) (at 142.24 135.89 90))
     (property "Value" "Conn_01x06" (id 1) (at 142.24 138.43 90))
     (property "Footprint" "Connector_PinHeader_2.54mm:PinHeader_1x06_P2.54mm_Horizontal" (id 2) (at 143.51 132.08 0)
@@
       (reference "A2") (unit 1) (value "GY-302_BH1750") (footprint "")
     )
+    (path "/421acf1c-f4d2-4059-83d6-dfb83d6549e9"
+      (reference "R1_GBR-618") (unit 1) (value "14.4R") (footprint "")
+    )
     (path "/d77d54ed-c281-49b8-a660-428ecc3d5c70"
-      (reference "J1") (unit 1) (value "Conn_01x06") (footprint "Connector_PinHeader_2.54mm:PinHeader_1x06_P2.54mm_Horizontal")
-    )
-    (path "/421acf1c-f4d2-4059-83d6-dfb83d6549e9"
-      (reference "R1") (unit 1) (value "GBR618") (footprint "")
+      (reference "X1") (unit 1) (value "Conn_01x06") (footprint "Connector_PinHeader_2.54mm:PinHeader_1x06_P2.54mm_Horizontal")
     )
   )
